Commit message: rviz+vision

File: src/agx_arm_moveit/config/agx_arm.srdf.xacro (robot description, xacro)
@@ -351,10 +351,10 @@
     <group_state name="home" group="arm">
       <joint name="joint1" value="0" />
-      <joint name="joint2" value="0" />
-      <joint name="joint3" value="0" />
-      <joint name="joint4" value="0" />
+      <joint name="joint2" value="0.8" />
+      <joint name="joint3" value="-1.2" />
+      <joint name="joint4" value="1.2" />
       <joint name="joint5" value="0" />
-      <joint name="joint6" value="0" />
-      <joint name="joint7" value="0" />
+      <joint name="joint6" value="-0.65" />
+      <joint name="joint7" value="0.6" />
     </group_state>
   </xacro:if>

Commit message: single_arm+single_grisp

File: src/agx_arm_moveit/config/agx_arm.srdf.xacro (robot description, xacro)
@@ -351,10 +351,10 @@
     <group_state name="home" group="arm">
       <joint name="joint1" value="0" />
-      <joint name="joint2" value="0.8" />
-      <joint name="joint3" value="-1.2" />
-      <joint name="joint4" value="1.2" />
+      <joint name="joint2" value="-0.390" />
+      <joint name="joint3" value="0.009" />
+      <joint name="joint4" value="2.147" />
       <joint name="joint5" value="0" />
-      <joint name="joint6" value="-0.65" />
-      <joint name="joint7" value="0.6" />
+      <joint name="joint6" value="0" />
+      <joint name="joint7" value="0.903" />
     </group_state>
   </xacro:if>

File: src/agx_arm_moveit/config/agx_arm.urdf.xacro (robot description, xacro)
@@ -7,6 +7,6 @@
   <xacro:arg name="tcp_offset_xyz" default="0 0 0" />
   <xacro:arg name="tcp_offset_rpy" default="0 0 0" />
-  <xacro:arg name="camera_mount_xyz" default="0.05 -0.04 0.06" />
-  <xacro:arg name="camera_mount_rpy" default="0 0.3 0" />
+  <xacro:arg name="camera_mount_xyz" default="0.0585 0.0 -0.0225" />
+  <xacro:arg name="camera_mount_rpy" default="0 0 -1.5708" />
   <xacro:property name="arm_type" value="$(arg arm_type)" />
   <xacro:property name="flange_link" value="${'link7' if arm_type == 'nero' else 'link6'}" />
@@ -26,7 +26,7 @@
   <link name="tcp_link" />
   <joint name="tcp_joint" type="fixed">
-    <parent link="${flange_link}" />
+    <parent link="gripper_link" />
     <child link="tcp_link" />
-    <origin xyz="$(arg tcp_offset_xyz)" rpy="$(arg tcp_offset_rpy)" />
+    <origin xyz="0 0 0.01" rpy="0 0 0" />
   </joint>
   <!-- Nominal wrist camera mount. Replace with calibrated hand-eye extrinsics. -->
@@ -38,5 +38,5 @@
   </link>
   <joint name="camera_mount_joint" type="fixed">
-    <parent link="${flange_link}" />
+    <parent link="gripper_link" />
     <child link="camera_link" />
     <origin xyz="$(arg camera_mount_xyz)" rpy="$(arg camera_mount_rpy)" />
@@ -46,5 +46,5 @@
     <parent link="camera_link" />
     <child link="camera_color_optical_frame" />
-    <origin xyz="0 0 0" rpy="-1.5708 0 -1.5708" />
+    <origin xyz="0.035 0 -0.055" rpy="0 0 0" />
   </joint>
   <xacro:include filename="agx_arm.ros2_control.xacro" />

Commit message: new pos

File: src/agx_arm_moveit/config/agx_arm.srdf.xacro (robot description, xacro)
@@ -350,11 +350,11 @@
   <xacro:if value="$(eval arm_type == 'nero')">
     <group_state name="home" group="arm">
-      <joint name="joint1" value="0" />
-      <joint name="joint2" value="-0.390" />
-      <joint name="joint3" value="0.009" />
-      <joint name="joint4" value="2.147" />
-      <joint name="joint5" value="0" />
-      <joint name="joint6" value="0" />
-      <joint name="joint7" value="0.903" />
+      <joint name="joint1" value="-1.751" />
+      <joint name="joint2" value="-0.342" />
+      <joint name="joint3" value="1.656" />
+      <joint name="joint4" value="1.036" />
+      <joint name="joint5" value="0.360" />
+      <joint name="joint6" value="0.074" />
+      <joint name="joint7" value="1.570" />
     </group_state>
   </xacro:if>

Commit message: fix_frame

File: src/agx_arm_moveit/config/agx_arm.srdf.xacro (robot description, xacro)
@@ -350,11 +350,11 @@
   <xacro:if value="$(eval arm_type == 'nero')">
     <group_state name="home" group="arm">
-      <joint name="joint1" value="-1.751" />
-      <joint name="joint2" value="-0.342" />
-      <joint name="joint3" value="1.656" />
-      <joint name="joint4" value="1.036" />
-      <joint name="joint5" value="0.360" />
-      <joint name="joint6" value="0.074" />
-      <joint name="joint7" value="1.570" />
+      <joint name="joint1" value="-0.0259" />
+      <joint name="joint2" value="-0.4025" />
+      <joint name="joint3" value="-0.0575" />
+      <joint name="joint4" value="2.1947" />
+      <joint name="joint5" value="0.0604" />
+      <joint name="joint6" value="0.0722" />
+      <joint name="joint7" value="0.9141" />
     </group_state>
   </xacro:if>

Commit message: fixframe1

File: src/agx_arm_moveit/config/agx_arm.srdf.xacro (robot description, xacro)
@@ -353,5 +353,5 @@
       <joint name="joint2" value="-0.4025" />
       <joint name="joint3" value="-0.0575" />
-      <joint name="joint4" value="2.1947" />
+      <joint name="joint4" value="2.0" />
       <joint name="joint5" value="0.0604" />
       <joint name="joint6" value="0.0722" />
