Commit message: rviz+virtual

File: src/agx_arm_moveit/config/agx_arm.urdf.xacro (robot description, xacro)
@@ -7,4 +7,6 @@
   <xacro:arg name="tcp_offset_xyz" default="0 0 0" />
   <xacro:arg name="tcp_offset_rpy" default="0 0 0" />
+  <xacro:arg name="camera_mount_xyz" default="0.05 -0.04 0.06" />
+  <xacro:arg name="camera_mount_rpy" default="0 0.3 0" />
   <xacro:property name="arm_type" value="$(arg arm_type)" />
   <xacro:property name="flange_link" value="${'link7' if arm_type == 'nero' else 'link6'}" />
@@ -28,4 +30,22 @@
     <origin xyz="$(arg tcp_offset_xyz)" rpy="$(arg tcp_offset_rpy)" />
   </joint>
+  <!-- Nominal wrist camera mount. Replace with calibrated hand-eye extrinsics. -->
+  <link name="camera_link">
+    <visual>
+      <geometry><box size="0.09 0.025 0.025" /></geometry>
+      <material name="camera_black"><color rgba="0.1 0.1 0.1 1" /></material>
+    </visual>
+  </link>
+  <joint name="camera_mount_joint" type="fixed">
+    <parent link="${flange_link}" />
+    <child link="camera_link" />
+    <origin xyz="$(arg camera_mount_xyz)" rpy="$(arg camera_mount_rpy)" />
+  </joint>
+  <link name="camera_color_optical_frame" />
+  <joint name="camera_to_color_optical" type="fixed">
+    <parent link="camera_link" />
+    <child link="camera_color_optical_frame" />
+    <origin xyz="0 0 0" rpy="-1.5708 0 -1.5708" />
+  </joint>
   <xacro:include filename="agx_arm.ros2_control.xacro" />
   <xacro:agx_arm_ros2_control

Commit message: camerapointcloud

File: src/agx_arm_moveit/config/agx_arm.urdf.xacro (robot description, xacro)
@@ -8,5 +8,5 @@
   <xacro:arg name="tcp_offset_rpy" default="0 0 0" />
   <xacro:arg name="camera_mount_xyz" default="0.0585 0.0 -0.0225" />
-  <xacro:arg name="camera_mount_rpy" default="0 0 -1.5708" />
+  <xacro:arg name="camera_mount_rpy" default="-1.5708 0 -1.5708" />
   <xacro:property name="arm_type" value="$(arg arm_type)" />
   <xacro:property name="flange_link" value="${'link7' if arm_type == 'nero' else 'link6'}" />
@@ -46,5 +46,5 @@
     <parent link="camera_link" />
     <child link="camera_color_optical_frame" />
-    <origin xyz="0.035 0 -0.055" rpy="0 0 0" />
+    <origin xyz="0.035 0 -0.055" rpy="-1.5708 0 -1.5708" />
   </joint>
   <xacro:include filename="agx_arm.ros2_control.xacro" />

Commit message: better path

File: src/agx_arm_moveit/config/agx_arm.urdf.xacro (robot description, xacro)
@@ -8,5 +8,5 @@
   <xacro:arg name="tcp_offset_rpy" default="0 0 0" />
   <xacro:arg name="camera_mount_xyz" default="0.0585 0.0 -0.0225" />
-  <xacro:arg name="camera_mount_rpy" default="-1.5708 0 -1.5708" />
+  <xacro:arg name="camera_mount_rpy" default="0 0 -1.5708" />
   <xacro:property name="arm_type" value="$(arg arm_type)" />
   <xacro:property name="flange_link" value="${'link7' if arm_type == 'nero' else 'link6'}" />
@@ -46,5 +46,5 @@
     <parent link="camera_link" />
     <child link="camera_color_optical_frame" />
-    <origin xyz="0.035 0 -0.055" rpy="-1.5708 0 -1.5708" />
+    <origin xyz="-0.035 0 0" rpy="0 0 0" />
   </joint>
   <xacro:include filename="agx_arm.ros2_control.xacro" />

Commit message: pos_fix

File: src/agx_arm_moveit/config/agx_arm.urdf.xacro (robot description, xacro)
@@ -46,5 +46,5 @@
     <parent link="camera_link" />
     <child link="camera_color_optical_frame" />
-    <origin xyz="-0.035 0 0" rpy="0 0 0" />
+    <origin xyz="0 0 0" rpy="0 0 3.1416" />
   </joint>
   <xacro:include filename="agx_arm.ros2_control.xacro" />

Commit message: statemachine update fix tcp_pos

File: src/agx_arm_moveit/config/agx_arm.urdf.xacro (robot description, xacro)
@@ -26,7 +26,7 @@
   <link name="tcp_link" />
   <joint name="tcp_joint" type="fixed">
-    <parent link="gripper_link" />
+    <parent link="gripper_base" />
     <child link="tcp_link" />
-    <origin xyz="0 0 0.01" rpy="0 0 0" />
+    <origin xyz="0 0 0.11" rpy="0 0 0" />
   </joint>
   <!-- Nominal wrist camera mount. Replace with calibrated hand-eye extrinsics. -->

Commit message: random_test

File: src/agx_arm_moveit/config/agx_arm.urdf.xacro (robot description, xacro)
@@ -7,5 +7,5 @@
   <xacro:arg name="tcp_offset_xyz" default="0 0 0" />
   <xacro:arg name="tcp_offset_rpy" default="0 0 0" />
-  <xacro:arg name="camera_mount_xyz" default="0.0585 0.0 -0.0225" />
+  <xacro:arg name="camera_mount_xyz" default="0.0585 0.0 0.0775" />
   <xacro:arg name="camera_mount_rpy" default="0 0 -1.5708" />
   <xacro:property name="arm_type" value="$(arg arm_type)" />
@@ -38,5 +38,5 @@
   </link>
   <joint name="camera_mount_joint" type="fixed">
-    <parent link="gripper_link" />
+    <parent link="gripper_base" />
     <child link="camera_link" />
     <origin xyz="$(arg camera_mount_xyz)" rpy="$(arg camera_mount_rpy)" />

Commit message: pos_fix!!!

File: src/agx_arm_moveit/config/agx_arm.urdf.xacro (robot description, xacro)
@@ -28,5 +28,5 @@
     <parent link="gripper_base" />
     <child link="tcp_link" />
-    <origin xyz="0 0 0.11" rpy="0 0 0" />
+    <origin xyz="0 0 0.11" rpy="0 0 3.1416" />
   </joint>
   <!-- Nominal wrist camera mount. Replace with calibrated hand-eye extrinsics. -->

Commit message: fixed_whole

File: src/agx_arm_moveit/config/agx_arm.urdf.xacro (robot description, xacro)
@@ -28,5 +28,5 @@
     <parent link="gripper_base" />
     <child link="tcp_link" />
-    <origin xyz="0 0 0.11" rpy="0 0 3.1416" />
+    <origin xyz="0 0 0.11" rpy="0 0 1.5708" />
   </joint>
   <!-- Nominal wrist camera mount. Replace with calibrated hand-eye extrinsics. -->

Commit message: fixed

File: src/agx_arm_moveit/config/agx_arm.urdf.xacro (robot description, xacro)
@@ -7,5 +7,5 @@
   <xacro:arg name="tcp_offset_xyz" default="0 0 0" />
   <xacro:arg name="tcp_offset_rpy" default="0 0 0" />
-  <xacro:arg name="camera_mount_xyz" default="0.0585 0.0 0.0775" />
+  <xacro:arg name="camera_mount_xyz" default="0.0585 0.0 0.0575" />
   <xacro:arg name="camera_mount_rpy" default="0 0 -1.5708" />
   <xacro:property name="arm_type" value="$(arg arm_type)" />
@@ -46,5 +46,5 @@
     <parent link="camera_link" />
     <child link="camera_color_optical_frame" />
-    <origin xyz="0 0 0" rpy="0 0 3.1416" />
+    <origin xyz="0.03 0 0" rpy="0 0 3.1416" />
   </joint>
   <xacro:include filename="agx_arm.ros2_control.xacro" />

Commit message: 夹取再优化

File: src/agx_arm_moveit/config/agx_arm.urdf.xacro (robot description, xacro)
@@ -28,5 +28,5 @@
     <parent link="gripper_base" />
     <child link="tcp_link" />
-    <origin xyz="0 0 0.11" rpy="0 0 1.5708" />
+    <origin xyz="0 0 0.135" rpy="0 0 1.5708" />
   </joint>
   <!-- Nominal wrist camera mount. Replace with calibrated hand-eye extrinsics. -->

Commit message: 强化学习+手动指令奖励

File: src/agx_arm_moveit/config/agx_arm.urdf.xacro (robot description, xacro)
@@ -28,5 +28,5 @@
     <parent link="gripper_base" />
     <child link="tcp_link" />
-    <origin xyz="0 0 0.135" rpy="0 0 1.5708" />
+    <origin xyz="0 0 0.12" rpy="0 0 1.5708" />
   </joint>
   <!-- Nominal wrist camera mount. Replace with calibrated hand-eye extrinsics. -->
